File: s.kicad_sch (KiCad schematic)
At the start: 0 parts

Commit message: got basic MCU powering from USBC
Parts:
- added C1, C3: 1uF, symbol Device:C_Small
- added C2, C6: 10uF, symbol Device:C_Small
- added C4, C5: 0.1uF, symbol Device:C_Small
- added J1: USB4085-GF-A_REVB, USB4085_GF_A:GCT_USB4085-GF-A_REVB, symbol USB4085-GF-A_REVB:USB4085-GF-A_REVB
- added R1: 10k, symbol Device:R_Small_US
- added U1: ESP32-S3-WROOM-1, RF_Module:ESP32-S3-WROOM-1, symbol RF_Module:ESP32-S3-WROOM-1
- added U2: MCP1825S, Package_TO_SOT_SMD:SOT-223-3_TabPin2, symbol Regulator_Linear:MCP1825S
Connections:
- new net: C1.1, R1.2, U1.3 (EN)
- new net +3.3V: C3.1, C5.1, C6.1, R1.1, U1.2 (3V3), U2.3 (VO)
- new net CC1: J1.A5 (CC1), U1.8 (IO15)
- new net CC2: J1.B5 (CC2), U1.9 (IO16)
- new net GND: C1.2, C2.2, C3.2, C4.2, C5.2, C6.2, J1.A1 (GND), J1.A12 (GND__1), J1.B1 (GND__2), J1.B12 (GND__3), J1.S1 (SHELL), J1.S2 (SHELL__1), J1.S3 (SHELL__2), J1.S4 (SHELL__3), U1.1 (GND), U1.40 (GND), U1.41 (GND), U2.2 (GND)
- new net USB_D+: J1.A6 (DP1), J1.B6 (DP2), U1.14 (USB_D+)
- new net USB_D-: J1.A7 (DN1), J1.B7 (DN2), U1.13 (USB_D-)
- new net VBUS: C2.1, C4.1, J1.A4 (VBUS), J1.A9 (VBUS__1), J1.B4 (VBUS__2), J1.B9 (VBUS__3), U2.1 (VI)
Other:
- added sheet switch_matrix (switch_matrix.kicad_sch)

Commit message: make key matrix
Other:
- sheet switch_matrix ports: added Col1, Col10, Col2, Col3, Col4, Col5, Col6, Col7, Col8, Col9, Row1, Row2, Row3; removed none
Changed lines of the file:
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@@
 	)
 	(sheet
-		(at 42.545 132.715)
-		(size 12.7 12.065)
+		(at 57.785 108.585)
+		(size 20.32 73.66)
 		(exclude_from_sim no)
 		(in_bom yes)
@@
 		)
 		(property "Sheetname" "switch_matrix"
-			(at 42.545 132.0034 0)
+			(at 57.785 107.8734 0)
 			(effects
 				(font
@@
 		)
 		(property "Sheetfile" "switch_matrix.kicad_sch"
-			(at 42.545 145.3646 0)
+			(at 57.785 182.8296 0)
 			(effects
 				(font
@@
 			)
 		)
+		(pin "Col1" bidirectional
+			(at 57.785 112.395 180)
+			(effects
+				(font
+					(size 1.27 1.27)
+				)
+				(justify left)
+			)
+		)
+		(pin "Col2" bidirectional
+			(at 57.785 116.205 180)
+			(effects
+				(font
+					(size 1.27 1.27)
+				)
+				(justify left)
+			)
+		)
+		(pin "Col3" bidirectional
+			(at 57.785 120.015 180)
+			(effects
+				(font
+					(size 1.27 1.27)
+				)
+				(justify left)
+			)
+		)
+		(pin "Col4" bidirectional
+			(at 57.785 123.825 180)
+			(effects
+				(font
+					(size 1.27 1.27)
+				)
+				(justify left)
+			)
+		)
+		(pin "Col5" bidirectional
+			(at 57.785 127.635 180)
+			(effects
+				(font
+					(size 1.27 1.27)
+				)
+				(justify left)
+			)
+		)
+		(pin "Col6" bidirectional
+			(at 57.785 131.445 180)
+			(effects
+				(font
+					(size 1.27 1.27)
+				)
+				(justify left)
+			)
+		)
+		(pin "Col7" bidirectional
+			(at 57.785 136.525 180)
+			(effects
+				(font
+					(size 1.27 1.27)
+				)
+				(justify left)
+			)
+		)
+		(pin "Col8" bidirectional
+			(at 57.785 139.7 180)
+			(effects
+				(font
+					(size 1.27 1.27)
+				)
+				(justify left)
+			)
+		)
+		(pin "Col9" bidirectional
+			(at 57.785 142.24 180)
+			(effects
+				(font
+					(size 1.27 1.27)
+				)
+				(justify left)
+			)
+		)
+		(pin "Col10" bidirectional
+			(at 57.785 144.78 180)
+			(effects
+				(font
+					(size 1.27 1.27)
+				)
+				(justify left)
+			)
+		)
+		(pin "Row1" bidirectional
+			(at 57.785 153.035 180)
+			(effects
+				(font
+					(size 1.27 1.27)
+				)
+				(justify left)
+			)
+		)
+		(pin "Row2" bidirectional
+			(at 57.785 155.575 180)
+			(effects
+				(font
+					(size 1.27 1.27)
+				)
+				(justify left)
+			)
+		)
+		(pin "Row3" bidirectional
+			(at 57.785 158.115 180)
+			(effects
+				(font
+					(size 1.27 1.27)
+				)
+				(justify left)
+			)
+		)
