File: switch_matrix.kicad_sch (KiCad schematic)
At the start: 0 parts

Commit message: make key matrix
Parts:
- added D1, D10, D11, D12, D13, D14, D15, D16, D17, D18, D19, D2, D20, D21, D22, D23, D24, D25, D3, D4, D5, D6, D7, D8, D9: ~, symbol Device:D_Small
- added SW1, SW20: Z, symbol Switch:SW_Push
- added SW10: D, symbol Switch:SW_Push
- added SW11, SW19: S, symbol Switch:SW_Push
- added SW12: K, symbol Switch:SW_Push
- added SW13: W, symbol Switch:SW_Push
- added SW14, SW16: R, symbol Switch:SW_Push
- added SW15, SW5: STAR, symbol Switch:SW_Push
- added SW17: B, symbol Switch:SW_Push
- added SW18: G, symbol Switch:SW_Push
- added SW2, SW9: T, symbol Switch:SW_Push
- added SW21: A, symbol Switch:SW_Push
- added SW22: O, symbol Switch:SW_Push
- added SW23: NUM, symbol Switch:SW_Push
- added SW24: E, symbol Switch:SW_Push
- added SW25: U, symbol Switch:SW_Push
- added SW3, SW7: P, symbol Switch:SW_Push
- added SW4: H, symbol Switch:SW_Push
- added SW6: F, symbol Switch:SW_Push
- added SW8: L, symbol Switch:SW_Push
Connections:
- new net: D24.2 (A), SW24.1
- new net: D1.2 (A), SW1.1
- new net: D17.2 (A), SW17.1
- new net: D4.2 (A), SW4.1
- new net: D10.2 (A), SW10.1
- new net: D23.2 (A), SW23.1
- new net: D19.2 (A), SW19.1
- new net: D12.2 (A), SW12.1
- new net: D16.2 (A), SW16.1
- new net: D22.2 (A), SW22.1
- new net: D13.2 (A), SW13.1
- new net: D3.2 (A), SW3.1
- new net: D8.2 (A), SW8.1
- new net: D15.2 (A), SW15.1
- new net: D9.2 (A), SW9.1
- new net: D21.2 (A), SW21.1
- new net: D2.2 (A), SW2.1
- new net: D7.2 (A), SW7.1
- new net: D20.2 (A), SW20.1
- new net: D5.2 (A), SW5.1
- new net: D14.2 (A), SW14.1
- new net: D6.2 (A), SW6.1
- new net: D18.2 (A), SW18.1
- new net: D25.2 (A), SW25.1
- new net: D11.2 (A), SW11.1
- new net Col1: SW1.2, SW11.2
- new net Col10: SW10.2, SW20.2
- new net Col2: SW12.2, SW2.2
- new net Col3: SW13.2, SW21.2, SW3.2
- new net Col4: SW14.2, SW22.2, SW4.2
- new net Col5: SW15.2, SW23.2, SW5.2
- new net Col6: SW16.2, SW24.2, SW6.2
- new net Col7: SW17.2, SW25.2, SW7.2
- new net Col8: SW18.2, SW8.2
- new net Col9: SW19.2, SW9.2
- new net Row1: D1.1 (K), D10.1 (K), D2.1 (K), D3.1 (K), D4.1 (K), D5.1 (K), D6.1 (K), D7.1 (K), D8.1 (K), D9.1 (K)
- new net Row2: D11.1 (K), D12.1 (K), D13.1 (K), D14.1 (K), D15.1 (K), D16.1 (K), D17.1 (K), D18.1 (K), D19.1 (K), D20.1 (K)
- new net Row3: D21.1 (K), D22.1 (K), D23.1 (K), D24.1 (K), D25.1 (K)
