File: battery_mgmt.kicad_sch (KiCad schematic)
At the start: 18 parts, among them J3 SW_PWR, J4 Conn_01x02_Pin, U3 MCP1825S, U4 AP9101CK, U5 MCP73831-2-OT, U6 DMG6968U-7, U7 DMG6968U-7

Commit message: update footprints
Parts:
- D30: footprint (none) -> LED_SMD:LED_0805_2012Metric_Pad1.15x1.40mm_HandSolder
- U6, U7: footprint DMG6968U-7:SOT95P240X110-3N -> DMG6968U_7:SOT95P240X110-3N
Changed lines of the file:
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@@
 			)
 		)
-		(property "Footprint" "DMG6968U-7:SOT95P240X110-3N"
+		(property "Footprint" "DMG6968U_7:SOT95P240X110-3N"
 			(at 167.64 116.84 0)
 			(effects
@@
 			)
 		)
-		(property "Footprint" "DMG6968U-7:SOT95P240X110-3N"
+		(property "Footprint" "DMG6968U_7:SOT95P240X110-3N"
 			(at 116.84 115.57 0)
 			(effects
@@
 			)
 		)
-		(property "Footprint" ""
+		(property "Footprint" "LED_SMD:LED_0805_2012Metric_Pad1.15x1.40mm_HandSolder"
 			(at 236.22 63.5 90)
 			(effects

Commit message: route battery charging stuff
Connections:
- net batt_pos: now reaches J3.3 (Pin_3), J4.1 (Pin_1), R7.1, U5.3 (V_{BAT})
- net batt_neg: now reaches C11.2, J4.2 (Pin_2), U4.3 (VSS), U6.2 (S)
- net between_mosfets: now reaches U6.3 (D), U7.3 (D)
Changed lines of the file:
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@@
+		)
+	)
+	(label "batt_pos"
+		(at 97.79 72.39 0)
+		(effects
+			(font
+				(size 1.27 1.27)
+			)
+			(justify left bottom)
 		)
 	)
@@
 		(effects
 			(font
+				(size 1.27 1.27)
+			)
+			(justify left bottom)
+		)
+	)
+	(label "between_mosfets"
+		(at 185.42 105.41 0)
+		(effects
+			(font
+				(size 1.27 1.27)
+			)
+			(justify left bottom)
+		)
+	)
+	(label "batt_neg"
+		(at 97.79 76.2 0)
+		(effects
+			(font

Commit message: modify schematic: add switch between voltage regs
Connections:
- net +3.3V renamed 3v3_from_batt
Changed lines of the file:
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@@
-	)
-	(junction
-		(at 62.23 110.49)
-		(diameter 0)
-		(color 0 0 0 0)
 	)
 	(junction
@@
 			)
 			(justify right)
+		)
+	)
+	(hierarchical_label "3v3_from_batt"
+		(shape bidirectional)
+		(at 62.23 110.49 0)
+		(effects
+			(font
+				(size 1.27 1.27)
+			)
+			(justify left)
 		)
 	)
@@
 					(unit 1)
 				)
-			)
-		)
-	)
-	(symbol
-		(lib_id "power:+3.3V")
-		(at 62.23 110.49 0)
-		(unit 1)
-		(exclude_from_sim no)
-		(in_bom yes)
-		(on_board yes)
-		(dnp no)
-		(fields_autoplaced yes)
-		(property "Reference" "#PWR018"
-			(at 62.23 114.3 0)
-			(effects
-				(font
-					(size 1.27 1.27)
-				)
-				(hide yes)
-			)
-		)
-		(property "Value" "+3.3V"
-			(at 62.23 105.41 0)
-			(effects
-				(font
-					(size 1.27 1.27)
-				)
-			)
-		)
-		(property "Footprint" ""
-			(at 62.23 110.49 0)
-			(effects
-				(font
-					(size 1.27 1.27)
-				)
-				(hide yes)
-			)
-		)
-		(property "Datasheet" ""
-			(at 62.23 110.49 0)
-			(effects
-				(font
-					(size 1.27 1.27)
-				)
-				(hide yes)
-			)
-		)
-		(property "Description" "Power symbol creates a global label with name \"+3.3V\""
-			(at 62.23 110.49 0)
-			(effects
-				(font
-					(size 1.27 1.27)
-				)
-				(hide yes)
-			)
-		)
-		(pin "1"
-		)
-		(instances
-			(project ""
-				(path "/915d30bc-a319-49d8-8691-e2837c0e16bd/ca799660-53b5-478c-aa84-f24ff3444acf"
-					(reference "#PWR018")
-					(unit 1)
-				)

Commit message: add a voltage divider for battery voltage monitoring
Parts:
- added R12: 30k, Resistor_SMD:R_0805_2012Metric_Pad1.20x1.40mm_HandSolder, symbol Device:R_Small_US
- added R13: 7.5k, Resistor_SMD:R_0805_2012Metric_Pad1.20x1.40mm_HandSolder, symbol Device:R_Small_US
Connections:
- net GND: now also R13.2
- net HV_CHR: now also R12.1
- new net vbatt_mon: R12.2, R13.1

Commit message: change power switch
Parts:
- removed J3: SW_PWR, Connector_PinHeader_2.54mm:PinHeader_1x03_P2.54mm_Vertical, symbol Connector:Conn_01x03_Pin
- added SW27: 09.03290.01, power_switch:09.03290_EAO, symbol power_switch:09.03290.01
Connections:
- net HV_CHR: now also SW27.2
- net batt_pos: now also SW27.1
Changed lines of the file:
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@@
+	(wire
+		(pts
+			(xy 90.17 38.1) (xy 97.79 38.1)
+		)
+		(stroke
+			(width 0)
+			(type default)
+		)
+	)
 	(wire
 		(pts
@@
 	(wire
 		(pts
-			(xy 99.06 49.53) (xy 99.06 43.18)
-		)
-		(stroke
-			(width 0)
-			(type default)
-		)
-	)
-	(wire
-		(pts
 			(xy 97.79 64.77) (xy 100.33 64.77)
 		)
@@
 	(wire
 		(pts
-			(xy 91.44 49.53) (xy 99.06 49.53)
-		)
-		(stroke
-			(width 0)
-			(type default)
-		)
-	)
-	(wire
-		(pts
 			(xy 114.3 73.66) (xy 114.3 91.44)
 		)
@@
 	(wire
 		(pts
+			(xy 97.79 38.1) (xy 97.79 57.15)
+		)
+		(stroke
+			(width 0)
+			(type default)
+		)
+	)
+	(wire
+		(pts
 			(xy 26.67 110.49) (xy 34.29 110.49)
 		)
@@
 	(wire
 		(pts
-			(xy 97.79 52.07) (xy 97.79 57.15)
-		)
-		(stroke
-			(width 0)
-			(type default)
-		)
-	)
-	(wire
-		(pts
 			(xy 97.79 72.39) (xy 91.44 72.39)
 		)
@@
 		(pts
 			(xy 160.02 82.55) (xy 160.02 91.44)
-		)
-		(stroke
-			(width 0)
-			(type default)
-		)
-	)
-	(wire
-		(pts
-			(xy 91.44 52.07) (xy 97.79 52.07)
 		)
 		(stroke
@@
 	)
 	(label "HV_CHR"
-		(at 99.06 43.18 90)
+		(at 64.77 35.56 180)
 		(effects
 			(font
 				(size 1.27 1.27)
 			)
-			(justify left bottom)
+			(justify right bottom)
 		)
 	)
@@
 	)
 	(symbol
+		(lib_id "power_switch:09.03290.01")
+		(at 64.77 35.56 0)
+		(unit 1)
+		(exclude_from_sim no)
+		(in_bom yes)
+		(on_board yes)
+		(dnp no)
+		(fields_autoplaced yes)
+		(property "Reference" "SW27"
+			(at 77.47 27.94 0)
+			(effects
+				(font
+					(size 1.524 1.524)
+				)
+			)
+		)
+		(property "Value" "09.03290.01"
+			(at 77.47 30.48 0)
+			(effects
+				(font
+					(size 1.524 1.524)
+				)
+			)
+		)
+		(property "Footprint" "power_switch:09.03290_EAO"
+			(at 64.77 35.56 0)
+			(effects
+				(font
+					(size 1.27 1.27)
+					(italic yes)
+				)
+				(hide yes)
+			)
+		)
+		(property "Datasheet" "09.03290.01"
+			(at 64.77 35.56 0)
+			(effects
+				(font
+					(size 1.27 1.27)
+					(italic yes)
+				)
+				(hide yes)
+			)
+		)
+		(property "Description" ""
+			(at 64.77 35.56 0)
+			(effects
+				(font
+					(size 1.27 1.27)
+				)
+				(hide yes)
+			)
+		)
+		(pin "3"
+		)
+		(pin "2"
+		)
+		(pin "1"
+		)
+		(instances
+			(project ""
+				(path "/915d30bc-a319-49d8-8691-e2837c0e16bd/ca799660-53b5-478c-aa84-f24ff3444acf"
+					(reference "SW27")
+					(unit 1)
+				)
+			)
+		)
+	)
+	(symbol
 		(lib_id "Battery_Management:AP9101CK")
 		(at 132.08 73.66 270)
@@
 					(unit 1)
 				)
-			)
-		)
-	)
-	(symbol
-		(lib_id "Connector:Conn_01x03_Pin")
-		(at 86.36 49.53 0)
-		(unit 1)
-		(exclude_from_sim no)
-		(in_bom yes)
-		(on_board yes)
-		(dnp no)
-		(fields_autoplaced yes)
-		(property "Reference" "J3"
-			(at 86.995 41.91 0)
-			(effects
-				(font
-					(size 1.27 1.27)
-				)
-			)
-		)
-		(property "Value" "SW_PWR"
-			(at 86.995 44.45 0)
-			(effects
-				(font
-					(size 1.27 1.27)
-				)
-			)
-		)
-		(property "Footprint" "Connector_PinHeader_2.54mm:PinHeader_1x03_P2.54mm_Vertical"
-			(at 86.36 49.53 0)
-			(effects
-				(font
-					(size 1.27 1.27)
-				)
-				(hide yes)
-			)
-		)
-		(property "Datasheet" "~"
-			(at 86.36 49.53 0)
-			(effects
-				(font
-					(size 1.27 1.27)
-				)
-				(hide yes)
-			)
-		)
-		(property "Description" "Generic connector, single row, 01x03, script generated"
-			(at 86.36 49.53 0)
-			(effects
-				(font
-					(size 1.27 1.27)
-				)
-				(hide yes)
-			)
-		)
-		(pin "3"
-		)
-		(pin "1"
-		)
-		(pin "2"
-		)
-		(instances
-			(project ""
-				(path "/915d30bc-a319-49d8-8691-e2837c0e16bd/ca799660-53b5-478c-aa84-f24ff3444acf"
-					(reference "J3")
-					(unit 1)
-				)

Commit message: change footprint of JST connector. Vertical -> horizontal
Parts:
- J4: footprint Connector_JST:JST_PH_B2B-PH-K_1x02_P2.00mm_Vertical -> Connector_JST:JST_PH_S2B-PH-K_1x02_P2.00mm_Horizontal
Changed lines of the file:
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@@
 			)
 		)
-		(property "Footprint" "Connector_JST:JST_PH_B2B-PH-K_1x02_P2.00mm_Vertical"
+		(property "Footprint" "Connector_JST:JST_PH_S2B-PH-K_1x02_P2.00mm_Horizontal"
 			(at 86.36 72.39 0)
 			(effects

Commit message: add a test point for battery voltage
Parts:
- added J1: Conn_01x02_Pin, Connector_PinHeader_2.54mm:PinHeader_1x02_P2.54mm_Vertical, symbol Connector:Conn_01x02_Pin
Connections:
- net GND: now also J1.2 (Pin_2)
- net HV_CHR: now also J1.1 (Pin_1)
Changed lines of the file:
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@@
+	)
+	(junction
+		(at 38.1 74.93)
+		(diameter 0)
+		(color 0 0 0 0)
 	)
 	(junction
@@
 	)
 	(junction
+		(at 38.1 53.34)
+		(diameter 0)
+		(color 0 0 0 0)
+	)
+	(junction
 		(at 54.61 110.49)
 		(diameter 0)
@@
 	(wire
 		(pts
+			(xy 38.1 53.34) (xy 46.99 53.34)
+		)
+		(stroke
+			(width 0)
+			(type default)
+		)
+	)
+	(wire
+		(pts
 			(xy 26.67 110.49) (xy 26.67 115.57)
 		)
@@
 	(wire
 		(pts
+			(xy 46.99 53.34) (xy 46.99 52.07)
+		)
+		(stroke
+			(width 0)
+			(type default)
+		)
+	)
+	(wire
+		(pts
 			(xy 114.3 73.66) (xy 114.3 91.44)
 		)
@@
 	(wire
 		(pts
-			(xy 38.1 73.66) (xy 38.1 76.2)
+			(xy 38.1 73.66) (xy 38.1 74.93)
 		)
 		(stroke
@@
 	(wire
 		(pts
+			(xy 38.1 74.93) (xy 50.8 74.93)
+		)
+		(stroke
+			(width 0)
+			(type default)
+		)
+	)
+	(wire
+		(pts
 			(xy 31.75 66.04) (xy 38.1 66.04)
 		)
@@
 	(wire
 		(pts
+			(xy 46.99 52.07) (xy 55.88 52.07)
+		)
+		(stroke
+			(width 0)
+			(type default)
+		)
+	)
+	(wire
+		(pts
 			(xy 149.86 91.44) (xy 160.02 91.44)
 		)
@@
 	(wire
 		(pts
+			(xy 50.8 74.93) (xy 50.8 54.61)
+		)
+		(stroke
+			(width 0)
+			(type default)
+		)
+	)
+	(wire
+		(pts
 			(xy 54.61 120.65) (xy 62.23 120.65)
 		)
@@
 	(wire
 		(pts
+			(xy 50.8 54.61) (xy 55.88 54.61)
+		)
+		(stroke
+			(width 0)
+			(type default)
+		)
+	)
+	(wire
+		(pts
 			(xy 213.36 67.31) (xy 220.98 67.31)
 		)
@@
 		(pts
 			(xy 43.18 120.65) (xy 54.61 120.65)
+		)
+		(stroke
+			(width 0)
+			(type default)
+		)
+	)
+	(wire
+		(pts
+			(xy 38.1 74.93) (xy 38.1 76.2)
 		)
 		(stroke
@@
 					(unit 1)
 				)
+			)
+		)
+	)
+	(symbol
+		(lib_id "Connector:Conn_01x02_Pin")
+		(at 60.96 52.07 0)
+		(mirror y)
+		(unit 1)
+		(exclude_from_sim no)
+		(in_bom yes)
+		(on_board yes)
+		(dnp no)
+		(fields_autoplaced yes)
+		(property "Reference" "J1"
+			(at 62.23 52.0699 0)
+			(effects
+				(font
+					(size 1.27 1.27)
+				)
+				(justify right)
+			)
+		)
+		(property "Value" "Conn_01x02_Pin"
+			(at 62.23 54.6099 0)
+			(effects
+				(font
+					(size 1.27 1.27)
+				)
+				(justify right)
+			)
+		)
+		(property "Footprint" "Connector_PinHeader_2.54mm:PinHeader_1x02_P2.54mm_Vertical"
+			(at 60.96 52.07 0)
+			(effects
+				(font
+					(size 1.27 1.27)
+				)
+				(hide yes)
+			)
+		)
+		(property "Datasheet" "~"
+			(at 60.96 52.07 0)
+			(effects
+				(font
+					(size 1.27 1.27)
+				)
+				(hide yes)
+			)
+		)
+		(property "Description" "Generic connector, single row, 01x02, script generated"
+			(at 60.96 52.07 0)
+			(effects
+				(font
+					(size 1.27 1.27)
+				)
+				(hide yes)
+			)
+		)
+		(pin "1"
+		)
+		(pin "2"
+		)
+		(instances
+			(project ""
+				(path "/915d30bc-a319-49d8-8691-e2837c0e16bd/ca799660-53b5-478c-aa84-f24ff3444acf"
+					(reference "J1")
+					(unit 1)
+				)
